File: Godzilla_Shield/Godzilla_Shield.sch (KiCad schematic (older format))
At the start: 9 parts, among them J1 6V, J2 12V, J3 Linha_Esq, J4 Linha_Dir, J5 Obstaculo, J6 Motor_Esq, J7 Motor_Dir, J8 Ultrassom

Commit message: Adiciona a versão 2 da placa
Connections:
- wire segments 48 -> 56
Changed lines of the file:
@@
 EESchema Schematic File Version 4
+LIBS:Godzilla_Shield-cache
 EELAYER 26 0
 EELAYER END
@@
 Title "Godzilla Shield"
 Date "2018-11-15"
-Rev "1.0"
+Rev "2.0"
 Comp "Laboratory of Prototyping, Robotics and Optimization"
 Comment1 "Author: Wederson Silva"
@@
 L Connector:Conn_01x03_Male J7
 U 1 1 5BED6943
-P 9350 6350
-F 0 "J7" V 9200 6350 50  0000 L CNN
-F 1 "Motor_Dir" V 9300 6200 50  0000 L CNN
-F 2 "Pin_Headers:Pin_Header_Straight_1x03_Pitch2.54mm" H 9350 6350 50  0001 C CNN
-F 3 "~" H 9350 6350 50  0001 C CNN
-	1    9350 6350
+P 9900 6350
+F 0 "J7" V 9950 6500 50  0000 L CNN
+F 1 "Motor_Dir" V 9850 6200 50  0000 L CNN
+F 2 "Pin_Headers:Pin_Header_Straight_1x03_Pitch2.54mm" H 9900 6350 50  0001 C CNN
+F 3 "~" H 9900 6350 50  0001 C CNN
+	1    9900 6350
 	0    -1   -1   0
 $EndComp
@@
 L Connector:Conn_01x03_Male J6
 U 1 1 5BED6EAF
-P 8950 6350
-F 0 "J6" V 8800 6350 50  0000 L CNN
-F 1 "Motor_Esq" V 8900 6200 50  0000 L CNN
-F 2 "Pin_Headers:Pin_Header_Straight_1x03_Pitch2.54mm" H 8950 6350 50  0001 C CNN
-F 3 "~" H 8950 6350 50  0001 C CNN
-	1    8950 6350
+P 9500 6350
+F 0 "J6" V 9550 6500 50  0000 L CNN
+F 1 "Motor_Esq" V 9450 6200 50  0000 L CNN
+F 2 "Pin_Headers:Pin_Header_Straight_1x03_Pitch2.54mm" H 9500 6350 50  0001 C CNN
+F 3 "~" H 9500 6350 50  0001 C CNN
+	1    9500 6350
 	0    -1   -1   0
 $EndComp
@@
 L Connector:Conn_01x03_Male J5
 U 1 1 5BED6EDD
-P 8500 6350
-F 0 "J5" V 8350 6350 50  0000 L CNN
-F 1 "Obstaculo" V 8450 6200 50  0000 L CNN
-F 2 "Pin_Headers:Pin_Header_Straight_1x03_Pitch2.54mm" H 8500 6350 50  0001 C CNN
-F 3 "~" H 8500 6350 50  0001 C CNN
-	1    8500 6350
+P 9000 6350
+F 0 "J5" V 9050 6500 50  0000 L CNN
+F 1 "Obstaculo" V 8950 6200 50  0000 L CNN
+F 2 "Pin_Headers:Pin_Header_Straight_1x03_Pitch2.54mm" H 9000 6350 50  0001 C CNN
+F 3 "~" H 9000 6350 50  0001 C CNN
+	1    9000 6350
 	0    -1   -1   0
 $EndComp
@@
 U 1 1 5BED6F03
 P 7850 6350
-F 0 "J4" V 7700 6350 50  0000 L CNN
+F 0 "J4" V 7900 6500 50  0000 L CNN
 F 1 "Linha_Dir" V 7800 6200 50  0000 L CNN
 F 2 "Pin_Headers:Pin_Header_Straight_1x03_Pitch2.54mm" H 7850 6350 50  0001 C CNN
@@
 U 1 1 5BED6F2D
 P 7400 6350
-F 0 "J3" V 7250 6350 50  0000 L CNN
+F 0 "J3" V 7450 6500 50  0000 L CNN
 F 1 "Linha_Esq" V 7350 6200 50  0000 L CNN
 F 2 "Pin_Headers:Pin_Header_Straight_1x03_Pitch2.54mm" H 7400 6350 50  0001 C CNN
@@
 U 1 1 5BED71B3
 P 7200 5350
-F 0 "J2" H 7050 5250 50  0000 L CNN
-F 1 "12V" H 7000 5350 50  0000 L CNN
+F 0 "J2" H 7200 5150 50  0000 L CNN
+F 1 "12V" H 7200 5450 50  0000 L CNN
 F 2 "Pin_Headers:Pin_Header_Straight_1x02_Pitch2.54mm" H 7200 5350 50  0001 C CNN
 F 3 "~" H 7200 5350 50  0001 C CNN
@@
 U 1 1 5BED733A
 P 7200 4800
-F 0 "J1" H 7050 4700 50  0000 L CNN
-F 1 "6V" H 7050 4800 50  0000 L CNN
+F 0 "J1" H 7200 4650 50  0000 L CNN
+F 1 "6V" H 7200 4900 50  0000 L CNN
 F 2 "Pin_Headers:Pin_Header_Straight_1x02_Pitch2.54mm" H 7200 4800 50  0001 C CNN
 F 3 "~" H 7200 4800 50  0001 C CNN
@@
 L Connector:Conn_01x04_Male J8
 U 1 1 5BED74F3
-P 9950 5950
-F 0 "J8" H 10100 6250 50  0000 R CNN
-F 1 "Ultrassom" H 10250 6150 50  0000 R CNN
-F 2 "Pin_Headers:Pin_Header_Straight_1x04_Pitch2.54mm" H 9950 5950 50  0001 C CNN
-F 3 "~" H 9950 5950 50  0001 C CNN
-	1    9950 5950
-	-1   0    0    1
+P 8400 6350
+F 0 "J8" V 8450 6600 50  0000 R CNN
+F 1 "Ultrassom" V 8350 6500 50  0000 R CNN
+F 2 "Pin_Headers:Pin_Header_Straight_1x04_Pitch2.54mm" H 8400 6350 50  0001 C CNN
+F 3 "~" H 8400 6350 50  0001 C CNN
+	1    8400 6350
+	0    -1   -1   0
 $EndComp
 Wire Wire Line
@@
 Wire Wire Line
 	7850 5900 7850 6150
-Wire Wire Line
-	9050 5750 9050 6150
-Wire Wire Line
-	9350 5850 9750 5850
-Wire Wire Line
-	9150 5750 9150 5950
-Wire Wire Line
-	9150 5950 9450 5950
-Wire Wire Line
-	9450 5950 9450 6150
 Wire Wire Line
 	7400 5450 7550 5450
@@
 GND
 Wire Wire Line
-	8850 6150 8700 6150
-Wire Wire Line
-	9250 6150 9100 6150
-Text Label 9100 6150 0    50   ~ 0
-GND
-Text Label 8700 6150 0    50   ~ 0
-GND
-Wire Wire Line
-	9350 6150 9350 6050
-Wire Wire Line
-	9350 6050 9250 6050
-Wire Wire Line
-	8950 6150 8950 6050
-Wire Wire Line
-	8950 6050 8850 6050
-Text Label 9250 6050 0    50   ~ 0
+	9800 6150 9650 6150
+Text Label 9650 6150 0    50   ~ 0
+GND
+Wire Wire Line
+	9900 6150 9900 6050
+Wire Wire Line
+	9900 6050 9800 6050
+Wire Wire Line
+	9500 6150 9500 6050
+Wire Wire Line
+	9500 6050 9400 6050
+Text Label 9800 6050 0    50   ~ 0
 6V
-Text Label 8850 6050 0    50   ~ 0
+Text Label 9400 6050 0    50   ~ 0
 6V
 Wire Wire Line
@@
 NoConn ~ 9350 4750
 NoConn ~ 9450 4750
-Wire Wire Line
-	9500 5900 9500 5950
-Wire Wire Line
-	9500 5950 9750 5950
-Text Label 9550 5850 0    50   ~ 0
-TRIG
-Text Label 9550 5950 0    50   ~ 0
-ECHO
-Wire Wire Line
-	9750 5750 9750 5600
-Wire Wire Line
-	9750 5600 9950 5600
-Text Label 9800 5600 0    50   ~ 0
-5V
-Wire Wire Line
-	9750 6050 9550 6050
-Text Label 9550 6050 0    50   ~ 0
-GND
 NoConn ~ 8150 5750
 NoConn ~ 8250 5750
-NoConn ~ 8950 5750
 NoConn ~ 9450 5750
 Wire Wire Line
@@
 5V
 Text Label 7150 6000 0    50   ~ 0
-5V
-Wire Wire Line
-	8400 6150 8250 6150
-Text Label 8250 6150 0    50   ~ 0
-GND
-Wire Wire Line
-	8500 6150 8500 6000
-Wire Wire Line
-	8500 6000 8350 6000
-Text Label 8350 6000 0    50   ~ 0
 5V
 Wire Wire Line
@@
 Text Label 8750 5950 1    50   ~ 0
 ECHO
-NoConn ~ 9350 5750
 NoConn ~ 9250 5750
 Wire Wire Line
-	8550 6050 8600 6050
-Wire Wire Line
-	8600 6050 8600 6150
-Wire Wire Line
-	8550 5750 8550 6050
-Wire Wire Line
-	8650 5750 8650 6000
+	8650 5750 8650 5950
 Text Label 8650 5950 1    50   ~ 0
 TRIG
+Wire Wire Line
+	8400 6150 8400 5950
+Wire Wire Line
+	8400 5950 8650 5950
+Wire Wire Line
+	8500 6150 8500 6000
+Wire Wire Line
+	8500 6000 8750 6000
+Wire Wire Line
+	8300 6150 8300 6050
+Wire Wire Line
+	8300 6050 8150 6050
+Text Label 8150 6050 0    50   ~ 0
+5V
+NoConn ~ 8550 5750
+NoConn ~ 9350 5750
+Wire Wire Line
+	8600 6150 8750 6150
+Text Label 8600 6150 0    50   ~ 0
+GND
+Wire Wire Line
+	9100 6150 9200 6150
+Text Label 9100 6150 0    50   ~ 0
+5V
+Wire Wire Line
+	9000 6150 9000 6000
+Text Label 9050 6000 0    50   ~ 0
+GND
+Wire Wire Line
+	9400 6150 9300 6150
+Wire Wire Line
+	9300 6150 9300 6000
+Wire Wire Line
+	9000 6000 9300 6000
+Wire Wire Line
+	9600 6150 9600 5950
+Wire Wire Line
+	9600 5950 9250 5950
+Wire Wire Line
+	9250 5950 9250 5850
+Wire Wire Line
+	9250 5850 9050 5850
+Wire Wire Line
+	9050 5850 9050 5750
+Wire Wire Line
+	10000 6150 10000 5900
+Wire Wire Line
+	10000 5900 9300 5900
+Wire Wire Line
+	9300 5900 9300 5800
+Wire Wire Line
+	9300 5800 9150 5800
+Wire Wire Line
+	9150 5800 9150 5750
+Wire Wire Line
+	8900 6150 8900 5800
+Wire Wire Line
+	8900 5800 8950 5800
+Wire Wire Line
+	8950 5800 8950 5750
 NoConn ~ 8850 5750
 $EndSCHEMATC
